Commit message: Update Práctica 2

File: catkin_ws/src/hardware/robot_description/justina_simple.urdf (robot description, URDF)
Before this commit: robot justina, 37 links, 36 joints
Links:
- removed link wheel_left
- removed link wheel_right
Joints:
- removed joint wheel_left_connect
- removed joint wheel_right_connect
