Commit message: Cambio de coordenadas de camera origin

File: catkin_ws/src/hardware/robot_description/robotino.urdf (robot description, URDF)
Before this commit: robot robotino, 8 links, 7 joints
Joints:
- joint depth_camera_joint: origin xyz=0 0 0.25 rpy=-1.8708 0 -1.5708 -> xyz=5 2 1 rpy=-1.8708 0 -1.5708
- joint depth_camera_joint2: origin xyz=0 0 0.25 rpy=-1.8708 0 -1.5708 -> xyz=5 2 1 rpy=-1.8708 0 -1.5708

Commit message: Practica 2 cambios en archivos

File: catkin_ws/src/hardware/robot_description/robotino.urdf (robot description, URDF)
Before this commit: robot robotino, 8 links, 7 joints
Joints:
- removed joint laser_joint
- joint depth_camera_joint2: origin xyz=0 0 0.25 rpy=-1.8708 0 -1.5708 -> xyz=-1 10 0.25 rpy=-1.8708 0 -1.5708

Commit message: Entrega Practica 2

File: catkin_ws/src/hardware/robot_description/robotino.urdf (robot description, URDF)
Before this commit: robot robotino, 8 links, 7 joints
Links:
- removed link laser_link
Joints:
- removed joint laser_joint
- joint depth_camera_joint: origin xyz=0 0 0.25 rpy=-1.8708 0 -1.5708 -> xyz=1 5 .25 rpy=0 0 2

Commit message: Practica 3

File: catkin_ws/src/hardware/robot_description/robotino.urdf (robot description, URDF)
Before this commit: robot robotino, 8 links, 6 joints
Joints:
- added joint laser_joint: type fixed, parent base_link, child laser_link, origin xyz=0 0 0.3 rpy=0 0 0, axis 0 0 0
- joint depth_camera_joint2: origin xyz=-1 10 0.25 rpy=-1.8708 0 -1.5708 -> xyz=0 0 0.25 rpy=-1.8708 0 -1.5708

Commit message: Practica 4

File: catkin_ws/src/hardware/robot_description/robotino.urdf (robot description, URDF)
Before this commit: robot robotino, 8 links, 7 joints
Joints:
- joint depth_camera_joint: origin xyz=5 5 0.25 rpy=-1.8708 0 -1.5708 -> xyz=0 0 0.25 rpy=-1.8708 0 -1.5708

Commit message: Practicas 3 y 4

File: catkin_ws/src/hardware/robot_description/robotino.urdf (robot description, URDF)
Before this commit: robot robotino, 7 links, 6 joints
Links:
- added link laser_link
Joints:
- added joint laser_joint: type fixed, parent base_link, child laser_link, origin xyz=0 0 0.3 rpy=0 0 0, axis 0 0 0

Commit message: Cambio de parametros en costmap

File: catkin_ws/src/hardware/robot_description/robotino.urdf (robot description, URDF)
Before this commit: robot robotino, 8 links, 7 joints
Joints:
- joint depth_camera_joint: origin xyz=5 2 1 rpy=-1.8708 0 -1.5708 -> xyz=0 0 0.25 rpy=-1.8708 0 -1.5708
- joint depth_camera_joint2: origin xyz=5 2 1 rpy=-1.8708 0 -1.5708 -> xyz=0 0 0.25 rpy=-1.8708 0 -1.5708

Commit message: Se añaden archivos hechos en las prácticas y las modificaciones pertinentes hechas a los archivos para la elaboración del proyecto. Instrucciones para la ejecución del proyecto añadidas a readme.md

File: catkin_ws/src/hardware/robot_description/robotino.urdf (robot description, URDF)
Before this commit: robot robotino, 8 links, 7 joints
Joints:
- joint depth_camera_joint2: origin xyz=0 0 0.25 rpy=-1.8708 0 -1.5708 -> xyz=0 0 0.25 rpy=-35.8708 140 -22.5708
